File: Kicad Files/Christmas Card.sch (KiCad schematic (older format))
At the start: 34 parts, among them J1 ISP, SW1 PWR, SW2 SW_Push, SW3 SW_Push, U1 ATtiny84-20SSU

Commit message: Initial Software
Parts:
- BT1: symbol Device:Battery_Cell -> Christmas-Card-rescue:Battery_Cell-Device
- C1: symbol Device:C -> Christmas-Card-rescue:C-Device
- J1: symbol Connector_Generic:Conn_02x03_Odd_Even -> Christmas-Card-rescue:Conn_02x03_Odd_Even-Connector_Generic
- LED1, LED10, LED11, LED12, LED13, LED14, LED15, LED16, LED17, LED18, LED19, LED2, LED20, LED3, LED4, LED5, LED6, LED7, LED8, LED9: symbol Device:LED -> Christmas-Card-rescue:LED-Device
- R1, R2, R3, R4, R5, R6, R7: symbol Device:R -> Christmas-Card-rescue:R-Device
- SW1: symbol Switch:SW_DPDT_x2 -> Christmas-Card-rescue:SW_DPDT_x2-Switch
- SW2, SW3: symbol Switch:SW_Push -> Christmas-Card-rescue:SW_Push-Switch
- U1: symbol MCU_Microchip_ATtiny:ATtiny84-20SSU -> Christmas-Card-rescue:ATtiny84-20SSU-MCU_Microchip_ATtiny
Changed lines of the file:
@@
 $EndDescr
 $Comp
-L Device:Battery_Cell BT1
+L Christmas-Card-rescue:Battery_Cell-Device BT1
 U 1 1 5D8C1116
 P 2300 4300
@@
 $EndComp
 $Comp
-L MCU_Microchip_ATtiny:ATtiny84-20SSU U1
+L Christmas-Card-rescue:ATtiny84-20SSU-MCU_Microchip_ATtiny U1
 U 1 1 5D8C25CB
 P 4650 3100
@@
 $EndComp
 $Comp
-L Device:LED LED1
+L Christmas-Card-rescue:LED-Device LED1
 U 1 1 5D8C75A1
 P 6500 2750
@@
 $EndComp
 $Comp
-L Device:LED LED9
+L Christmas-Card-rescue:LED-Device LED9
 U 1 1 5D8CA536
 P 6500 3250
@@
 $EndComp
 $Comp
-L Device:LED LED15
+L Christmas-Card-rescue:LED-Device LED15
 U 1 1 5D8CA540
 P 6500 3750
@@
 $EndComp
 $Comp
-L Device:LED LED19
+L Christmas-Card-rescue:LED-Device LED19
 U 1 1 5D8CC876
 P 6500 4250
@@
 $EndComp
 $Comp
-L Device:LED LED2
+L Christmas-Card-rescue:LED-Device LED2
 U 1 1 5D8D51BA
 P 7000 2250
@@
 $EndComp
 $Comp
-L Device:LED LED3
+L Christmas-Card-rescue:LED-Device LED3
 U 1 1 5D8D51CE
 P 7000 3250
@@
 $EndComp
 $Comp
-L Device:LED LED11
+L Christmas-Card-rescue:LED-Device LED11
 U 1 1 5D8D51D8
 P 7000 3750
@@
 $EndComp
 $Comp
-L Device:LED LED17
+L Christmas-Card-rescue:LED-Device LED17
 U 1 1 5D8D51E2
 P 7000 4250
@@
 $EndComp
 $Comp
-L Device:LED LED10
+L Christmas-Card-rescue:LED-Device LED10
 U 1 1 5D8E7BD6
 P 7500 2250
@@
 $EndComp
 $Comp
-L Device:LED LED4
+L Christmas-Card-rescue:LED-Device LED4
 U 1 1 5D8E7BE0
 P 7500 2750
@@
 $EndComp
 $Comp
-L Device:LED LED5
+L Christmas-Card-rescue:LED-Device LED5
 U 1 1 5D8E7BF4
 P 7500 3750
@@
 $EndComp
 $Comp
-L Device:LED LED13
+L Christmas-Card-rescue:LED-Device LED13
 U 1 1 5D8E7BFE
 P 7500 4250
@@
 $EndComp
 $Comp
-L Device:LED LED16
+L Christmas-Card-rescue:LED-Device LED16
 U 1 1 5D8E7C12
 P 8000 2250
@@
 $EndComp
 $Comp
-L Device:LED LED12
+L Christmas-Card-rescue:LED-Device LED12
 U 1 1 5D8E7C1C
 P 8000 2750
@@
 $EndComp
 $Comp
-L Device:LED LED6
+L Christmas-Card-rescue:LED-Device LED6
 U 1 1 5D8E7C26
 P 8000 3250
@@
 $EndComp
 $Comp
-L Device:LED LED7
+L Christmas-Card-rescue:LED-Device LED7
 U 1 1 5D8E7C3A
 P 8000 4250
@@
 $EndComp
 $Comp
-L Device:LED LED20
+L Christmas-Card-rescue:LED-Device LED20
 U 1 1 5D8F04B0
 P 8500 2250
@@
 $EndComp
 $Comp
-L Device:LED LED18
+L Christmas-Card-rescue:LED-Device LED18
 U 1 1 5D8F04BA
 P 8500 2750
@@
 $EndComp
 $Comp
-L Device:LED LED14
+L Christmas-Card-rescue:LED-Device LED14
 U 1 1 5D8F04C4
 P 8500 3250
@@
 $EndComp
 $Comp
-L Device:LED LED8
+L Christmas-Card-rescue:LED-Device LED8
 U 1 1 5D8F04CE
 P 8500 3750
@@
 $EndComp
 $Comp
-L Device:R R1
+L Christmas-Card-rescue:R-Device R1
 U 1 1 5D8F8CC7
 P 6500 2250
@@
 $EndComp
 $Comp
-L Device:R R2
+L Christmas-Card-rescue:R-Device R2
 U 1 1 5D8FD82E
 P 7000 2750
@@
 $EndComp
 $Comp
-L Device:R R3
+L Christmas-Card-rescue:R-Device R3
 U 1 1 5D8FE06B
 P 7500 3250
@@
 $EndComp
 $Comp
-L Device:R R4
+L Christmas-Card-rescue:R-Device R4
 U 1 1 5D8FEC66
 P 8000 3750
@@
 $EndComp
 $Comp
-L Device:R R5
+L Christmas-Card-rescue:R-Device R5
 U 1 1 5D8FF4B0
 P 8500 4250
@@
 $EndComp
 $Comp
-L Switch:SW_Push SW2
+L Christmas-Card-rescue:SW_Push-Switch SW2
 U 1 1 5D90A757
 P 6850 5000
@@
 $EndComp
 $Comp
-L Switch:SW_Push SW3
+L Christmas-Card-rescue:SW_Push-Switch SW3
 U 1 1 5D90B010
 P 7850 5000
@@
 	8500 2500 8000 2500
 $Comp
-L power:+BATT #PWR0101
+L Christmas-Card-rescue:+BATT-power #PWR0101
 U 1 1 5DAB74AD
 P 2650 2900
@@
 $EndComp
 $Comp
-L power:+BATT #PWR0102
+L Christmas-Card-rescue:+BATT-power #PWR0102
 U 1 1 5DABE4FE
 P 7150 4900
@@
 $EndComp
 $Comp
-L power:+BATT #PWR0103
+L Christmas-Card-rescue:+BATT-power #PWR0103
 U 1 1 5DABEB7C
 P 8150 4900
@@
 	7150 5000 7150 4900
 $Comp
-L Device:R R7
+L Christmas-Card-rescue:R-Device R7
 U 1 1 5DAEAE80
 P 7500 5250
@@
 $EndComp
 $Comp
-L Device:R R6
+L Christmas-Card-rescue:R-Device R6
 U 1 1 5DAEB3B7
 P 6500 5250
@@
 	5750 4700 6500 4700
 $Comp
-L power:GND #PWR0104
+L Christmas-Card-rescue:GND-power #PWR0104
 U 1 1 5DC5D188
 P 6500 5500
@@
 $EndComp
 $Comp
-L power:GND #PWR0105
+L Christmas-Card-rescue:GND-power #PWR0105
 U 1 1 5DC5D608
 P 7500 5500
@@
 	6500 5500 6500 5400
 $Comp
-L power:GND #PWR0106
+L Christmas-Card-rescue:GND-power #PWR0106
 U 1 1 5DC8071B
 P 2300 4600
@@
 $EndComp
 $Comp
-L Device:C C1
+L Christmas-Card-rescue:C-Device C1
 U 1 1 5DCB1CE4
 P 3050 3750
@@
 	3050 3000 3050 3600
 $Comp
-L Connector_Generic:Conn_02x03_Odd_Even J1
+L Christmas-Card-rescue:Conn_02x03_Odd_Even-Connector_Generic J1
 U 1 1 5DCEB63D
 P 4700 5300
@@
 	5350 5300 5000 5300
 $Comp
-L power:GND #PWR0107
+L Christmas-Card-rescue:GND-power #PWR0107
 U 1 1 5DDD352C
 P 5250 5500
@@
 $EndComp
 $Comp
-L power:+BATT #PWR0108
+L Christmas-Card-rescue:+BATT-power #PWR0108
 U 1 1 5DDD396C
 P 5250 5050
@@
 	5250 5400 5250 5500
 $Comp
-L power:GND #PWR0109
+L Christmas-Card-rescue:GND-power #PWR0109
 U 1 1 5DDFB0E0
 P 4650 4100
@@
 $EndComp
 $Comp
-L power:+BATT #PWR0110
+L Christmas-Card-rescue:+BATT-power #PWR0110
 U 1 1 5DDFD2F3
 P 4650 2100
@@
 	6500 5000 6500 4700
 $Comp
-L Switch:SW_DPDT_x2 SW1
+L Christmas-Card-rescue:SW_DPDT_x2-Switch SW1
 U 1 1 5E0A6C1E
 P 2550 3300
@@
 $EndComp
 $Comp
-L Switch:SW_DPDT_x2 SW1
+L Christmas-Card-rescue:SW_DPDT_x2-Switch SW1
 U 2 1 5E0A7978
 P 2050 3300
@@
 	2300 4500 2300 4600
 $Comp
-L power:PWR_FLAG #FLG0101
+L Christmas-Card-rescue:PWR_FLAG-power #FLG0101
 U 1 1 5E144AF7
 P 3000 5600
@@
 $EndComp
 $Comp
-L power:PWR_FLAG #FLG0102
+L Christmas-Card-rescue:PWR_FLAG-power #FLG0102
 U 1 1 5E14903B
 P 2500 5500
@@
 $EndComp
 $Comp
-L power:GND #PWR0111
+L Christmas-Card-rescue:GND-power #PWR0111
 U 1 1 5E149A52
 P 2500 5600
@@
 $EndComp
 $Comp
-L power:+BATT #PWR0112
+L Christmas-Card-rescue:+BATT-power #PWR0112
 U 1 1 5E149FD7
 P 3000 5500
